File: PCB/programmable-air-v0.2/slave-board.brd (EAGLE design)
At the start: 97.7 x 49 mm, 37 parts, among them IC1 INA126U, IC3 LM358MX, Q1 600mA/40V, Q2 600mA/40V, Q3 600mA/40V

Commit message: LM358 slave board final
Parts:
- removed R10: 1.78K, eagle-ltspice:R0603
- removed R13, R14, R15, R8, R9: 10K, eagle-ltspice:R0603
- removed R16: 40K, eagle-ltspice:R0603
- removed R17, R20: 20K, eagle-ltspice:R0603
- added R11, R12, R18, R19, R4: 10k, SparkFun-Resistors:0603
- added R21: 40K, SparkFun-Resistors:0603
- added R22, R23: 20K, SparkFun-Resistors:0603
- added R24: 2K, SparkFun-Resistors:0603
- moved C2 9.16 mm to (6.35, 37.5), turned to 0 degrees
- moved C1 2.54 mm to (78.1, 36.8)
- moved D1 0.63 mm to (56.5, 5.08)
- moved D2 0.63 mm to (22.9, 5.08)
- moved D3 0.63 mm to (87.6, 5.08)
- moved U$1 0.63 mm to (50.2, 38.1)
Connections:
- new net N$16: IC1.6, R22.1
- net GND: now also R11.1, R12.1, R23.1, R4.1; no longer R14.1, R17.1, R8.1, R9.1
- net N$13: now also R19.1; no longer R13.1
- net N$15: now also R18.2, R21.1; no longer R15.2, R16.2, R20.2
- net N$24: now also R21.2, R4.2; no longer R16.1, R8.2
- net N$25: now also R24.1; no longer R10.1
- net N$26: now also R24.2; no longer R10.2
- net N$27: now also R19.2, R22.2, R23.2; no longer R13.2, R17.2, R20.1
- net N$30: now also R12.2, R18.1; no longer R14.2, R15.1
- net N$31: now also R11.2; no longer R9.2
Routing:
- net N$15: track 322.2 -> 275.3 mm
- net N$16: track 0.00 -> 46.1 mm
- net VIN: track 417.3 -> 397.2 mm, vias 3 -> 4
- net N$24: track 1.99 -> 9.51 mm
- net GND: track 51.6 -> 46.8 mm
- net N$8: track 15.4 -> 20.2 mm
- net N$7: track 20.1 -> 23.4 mm
- net N$13: track 97.5 -> 100.4 mm
- net N$30: track 7.13 -> 9.88 mm
- net N$31: track 17.0 -> 14.5 mm
- net N$19: track 35.5 -> 36.8 mm
- net N$1: track 37.2 -> 35.9 mm
- net N$2: track 39.9 -> 38.8 mm
- net N$6: track 6.53 -> 5.89 mm
- net N$18: track 7.16 -> 6.53 mm
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