File: PCB/programmable-air-v0.2/master-board plus slave.sch (EAGLE design)
At the start: 74 parts, among them IC2 INA126U, IC4 LM358MX, J1 POWER_JACKTOE, Q4 600mA/40V, Q5 600mA/40V, Q6 600mA/40V

Commit message: Sent PCBs for fabrication
Parts:
- added C10, C11: 0.1uF, SparkFun-Passives:CAP0603-CAP
- added R5, R7: (no value), SparkFun-Resistors:RESISTOR0603
- added R6, R8: (no value), SparkFun-Resistors:RESISTOR1206
- added U$10, U$11, U$12, U$9: FIDUCIAL, adafruit:FIDUCIAL
- added U1, U2: INA169, SparkFun-AnalogIC:INA169
- R34: value 40K -> 10k
- R35, R36: value 20K -> 10k
- R37: value 2K -> 10k
Connections:
- removed net N$64: J7.6, J8.6
- new net VIN-: D2.A, R6.2, U$2.P$1, U$4.P$1, U2.VIN-
- new net VIN-1: D1.A, R8.2, U$1.P$1, U$3.P$1, U1.VIN-
- new net VOUT: ARDUINO_NANO1.ADC6/A6, R7.2, U1.OUT
- new net VOUT1: ARDUINO_NANO1.ADC7/A7, R5.2, U2.OUT
- net GND: now also C10.1, C11.1, R5.1, R7.1, U1.GND, U2.GND
- net N$13: now also ARDUINO_NANO1.ADC2/A2; no longer ARDUINO_NANO1.ADC3/A3
- net N$14: now also ARDUINO_NANO1.ADC5/SCL/A5; no longer ARDUINO_NANO1.ADC4/SDA/A4
- net N$18: now also ARDUINO_NANO1.ADC4/SDA/A4; no longer ARDUINO_NANO1.ADC2/A2
- net N$63: now also ARDUINO_NANO1.ADC3/A3; no longer ARDUINO_NANO1.ADC5/SCL/A5
- net VCC: now also C10.2, C11.2, U1.V+, U2.V+
- net VIN: now also R6.1, R8.1, U1.VIN+, U2.VIN+; no longer D1.A, D2.A, U$1.P$1, U$2.P$1, U$3.P$1, U$4.P$1
Other:
- note added: "RS"
