File: PCB/programmable-air-v0.2/slave-board.sch (EAGLE design)
At the start: 37 parts, among them IC1 INA126U, IC3 LM358MX, Q1 600mA/40V, Q2 600mA/40V, Q3 600mA/40V

Commit message: Sent for second production run. New Logo.
Parts:
- removed R13, R14, R15: 10K, eagle-ltspice:RR0603
- removed R16: 40K, eagle-ltspice:RR0603
- removed R17, R20: 20K, eagle-ltspice:RR0603
- added C3, C4: 1.0uF, SparkFun-Capacitors:1.0UF-0603-16V-10%
- added C5: 22uF, SparkFun-Capacitors:22UF-POLAR-PANASONIC_C-35V-20%
- added R11, R12, R18, R19, R4: 10k, SparkFun-Resistors:10KOHM-0603-1/10W-1%
- added R21: 40K, SparkFun-Resistors:10KOHM-0603-1/10W-1%
- added R22, R23: 20K, SparkFun-Resistors:10KOHM-0603-1/10W-1%
- added R24: 2K, SparkFun-Resistors:10KOHM-0603-1/10W-1%
- R10: value 1.78K -> 1k; device eagle-ltspice:RR0603 -> SparkFun-Resistors:1KOHM-0603-1/10W-1%
- R8, R9: value 10K -> 1k; device eagle-ltspice:RR0603 -> SparkFun-Resistors:1KOHM-0603-1/10W-1%
Connections:
- removed net N$15: C1.+, IC1.REF, IC3P.V+, J1.7, J2.7, R15.2, R16.2, R20.2, U$10.P$1, U$8.P$1, U$9.P$1
- removed net VIN: C2.+, D1.A, D2.A, D3.A, IC1.V+, J1.1, J2.1, U$2.P$1, U$3.P$1, U$4.P$1, U$5.P$1, U$6.P$1, U$7.P$1
- new net N$16: IC1.OUT, R22.1
- new net N$17: C2.+, C4.1, C5.+, D1.A, D2.A, D3.A, IC1.V+, J1.1, J2.1, U$2.P$1, U$3.P$1, U$4.P$1, U$5.P$1, U$6.P$1, U$7.P$1
- new net N$21: R8.2, U$8.P$1
- new net N$22: R9.2, U$9.P$1
- new net N$23: R10.2, U$10.P$1
- new net N$28: C1.+, C3.1, IC1.REF, IC3P.V+, J1.7, J2.7, R10.1, R18.2, R21.1, R8.1, R9.1
- net GND: now also C3.2, C4.2, C5.-, R11.1, R12.1, R23.1, R4.1; no longer R14.1, R17.1, R8.1, R9.1
- net N$13: now also R19.1; no longer R13.1
- net N$24: now also R21.2, R4.2; no longer R16.1, R8.2
- net N$25: now also R24.1; no longer R10.1
- net N$26: now also R24.2; no longer R10.2
- net N$27: now also R19.2, R22.2, R23.2; no longer R13.2, R17.2, R20.1
- net N$30: now also R12.2, R18.1; no longer R14.2, R15.1
- net N$31: now also R11.2; no longer R9.2
Other:
- moved on the sheet: IC1, IC3A, IC3B
